File: PCB Sources/Monorail_Steam_Reduced/Monorail_Steam_Reduced.kicad_pcb (KiCad board)
At the start: 2 copper layers, 242.9 x 76.2 mm, 7 parts, among them J6 USB_C_Receptacle_USB2.0

Commit message: updated positions, readme, deleted unecessary files
Parts:
- removed the REF** at (242.5, 71.0)
- removed the REF** at (247.4, 69.7)
- removed the REF** at (237.6, 69.7)
- added C1: 10u, Capacitor_SMD:C_0402_1005Metric, B.Cu at (140.3, -23.6)
- added C10: 0.1uF, Capacitor_SMD:C_0603_1608Metric, B.Cu at (124.5, -56.1)
- added C11: 0.1uF, Capacitor_SMD:C_0603_1608Metric, B.Cu at (124.5, -53.5)
- added C12: 0.1uF, Capacitor_SMD:C_0603_1608Metric, B.Cu at (124.5, -51.0)
- added C13: 0.1uF, Capacitor_SMD:C_0603_1608Metric, B.Cu at (124.5, -48.5)
- added C14: 0.1uF, Capacitor_SMD:C_0603_1608Metric, B.Cu at (124.5, -46.0)
- added C15: 0.1uF, Capacitor_SMD:C_0603_1608Metric, B.Cu at (124.5, -43.5)
- added C16: 0.1uF, Capacitor_SMD:C_0603_1608Metric, B.Cu at (120.5, -58.6)
- added C17: 0.1uF, Capacitor_SMD:C_0603_1608Metric, B.Cu at (120.5, -56.1)
- added C18: 0.1uF, Capacitor_SMD:C_0603_1608Metric, B.Cu at (120.5, -53.5)
- added C19: 0.1uF, Capacitor_SMD:C_0603_1608Metric, B.Cu at (120.5, -51.0)
- added C2: 10u, Capacitor_SMD:C_0402_1005Metric, B.Cu at (140.3, -21.7)
- added C20: 0.1uF, Capacitor_SMD:C_0603_1608Metric, B.Cu at (120.5, -48.5)
- added C21: 100n, Capacitor_SMD:C_0402_1005Metric, B.Cu at (134.6, -23.6)
- added C22: 100n, Capacitor_SMD:C_0402_1005Metric, B.Cu at (134.6, -21.7)
- added C23: 100n, Capacitor_SMD:C_0402_1005Metric, B.Cu at (134.6, -19.7)
- added C24: 100n, Capacitor_SMD:C_0402_1005Metric, B.Cu at (134.6, -17.7)
- added C25: 100n, Capacitor_SMD:C_0402_1005Metric, B.Cu at (131.7, -23.6)
- added C26: 100n, Capacitor_SMD:C_0402_1005Metric, B.Cu at (131.7, -21.7)
- added C27: 30p, Capacitor_SMD:C_0402_1005Metric, B.Cu at (236.5, 97.4)
- added C28: 100n, Capacitor_SMD:C_0402_1005Metric, B.Cu at (131.7, -17.7)
- added C3: 1u, Capacitor_SMD:C_0402_1005Metric, B.Cu at (252.2, 98.9)
- added C4: 10u, Capacitor_SMD:C_0402_1005Metric, B.Cu at (252.3, 97.9)
- added C5: 1u, Capacitor_SMD:C_0402_1005Metric, B.Cu at (242.6, 94.9)
- added C6: 30p, Capacitor_SMD:C_0402_1005Metric, B.Cu at (236.5, 96.1)
- added C7: 100n, Capacitor_SMD:C_0402_1005Metric, B.Cu at (137.5, -19.7)
- added C8: 100n, Capacitor_SMD:C_0402_1005Metric, B.Cu at (137.5, -17.7)
- added C9: 0.1uF, Capacitor_SMD:C_0603_1608Metric, B.Cu at (124.5, -58.6)
- added D1: BAV70, Package_TO_SOT_SMD:SOT-23, B.Cu at (153.0, 162.7)
- added D10: BAV70, Package_TO_SOT_SMD:SOT-23, B.Cu at (139.6, 167.2)
- added D11: BAV70, Package_TO_SOT_SMD:SOT-23, B.Cu at (135.2, 167.2)
- added D12: BAV70, Package_TO_SOT_SMD:SOT-23, B.Cu at (130.7, 167.2)
- added D13: BAV70, Package_TO_SOT_SMD:SOT-23, B.Cu at (153.0, 171.8)
- added D14: BAV70, Package_TO_SOT_SMD:SOT-23, B.Cu at (148.5, 171.8)
- added D15: BAV70, Package_TO_SOT_SMD:SOT-23, B.Cu at (144.1, 171.8)
- added D16: BAV70, Package_TO_SOT_SMD:SOT-23, B.Cu at (139.6, 171.8)
- added D17: BAV70, Package_TO_SOT_SMD:SOT-23, B.Cu at (135.2, 171.8)
- added D18: BAV70, Package_TO_SOT_SMD:SOT-23, B.Cu at (130.7, 171.8)
- added D19: BAV70, Package_TO_SOT_SMD:SOT-23, B.Cu at (153.0, 176.3)
- added D2: BAV70, Package_TO_SOT_SMD:SOT-23, B.Cu at (148.5, 162.7)
- added D20: BAV70, Package_TO_SOT_SMD:SOT-23, B.Cu at (148.5, 176.3)
- added D21: BAV70, Package_TO_SOT_SMD:SOT-23, B.Cu at (144.1, 176.3)
- added D22: BAV70, Package_TO_SOT_SMD:SOT-23, B.Cu at (139.6, 176.3)
- added D3: BAV70, Package_TO_SOT_SMD:SOT-23, B.Cu at (144.1, 162.7)
- added D4: BAV70, Package_TO_SOT_SMD:SOT-23, B.Cu at (139.6, 162.7)
- added D5: BAV70, Package_TO_SOT_SMD:SOT-23, B.Cu at (135.2, 162.7)
- added D53: LED, LED_THT:LED_D3.0mm, B.Cu at (140.1, -38.5)
- added D54: LED, LED_THT:LED_D3.0mm, B.Cu at (140.1, -32.9)
- added D55: LED, LED_THT:LED_D3.0mm, B.Cu at (140.1, -27.4)
- added D56: WS2812B, WS2812B:WS2812B_data-bridgeable, B.Cu at (143.5, 96.4)
- added D57: WS2812B, WS2812B:WS2812B_data-bridgeable, B.Cu at (181.6, 96.4)
- added D58: WS2812B, WS2812B:WS2812B_data-bridgeable, B.Cu at (219.9, 96.4)
- added D59: WS2812B, WS2812B:WS2812B_data-bridgeable, B.Cu at (229.1, 115.6)
- added D6: BAV70, Package_TO_SOT_SMD:SOT-23, B.Cu at (130.7, 162.7)
- added D60: WS2812B, WS2812B:WS2812B_data-bridgeable, B.Cu at (191.3, 115.6)
- added D61: WS2812B, WS2812B:WS2812B_data-bridgeable, B.Cu at (152.9, 115.6)
- added D62: WS2812B, WS2812B:WS2812B_data-bridgeable, B.Cu at (115.0, 115.6)
- added D63: WS2812B, WS2812B:WS2812B_data-bridgeable, B.Cu at (95.9, 115.6)
- added D64: WS2812B, WS2812B:WS2812B_data-bridgeable, B.Cu at (105.6, 96.4)
- added D65: WS2812B, WS2812B:WS2812B_data-bridgeable, B.Cu at (86.5, 96.4)
- added D66: WS2812B, WS2812B:WS2812B_data-bridgeable, B.Cu at (67.3, 96.4)
- added D67: WS2812B, WS2812B:WS2812B_data-bridgeable, B.Cu at (76.9, 115.6)
- added D7: BAV70, Package_TO_SOT_SMD:SOT-23, B.Cu at (153.0, 167.2)
- added D8: BAV70, Package_TO_SOT_SMD:SOT-23, B.Cu at (148.5, 167.2)
- added D9: BAV70, Package_TO_SOT_SMD:SOT-23, B.Cu at (144.1, 167.2)
- added F1: 500mA, Fuse:Fuse_1206_3216Metric, B.Cu at (117.5, -15.1)
- added J8: Conn_01x04_Male, Connector_PinHeader_2.54mm:PinHeader_1x04_P2.54mm_Vertical, B.Cu at (124.0, -38.9)
- added J9: Conn_01x03_Male, Connector_PinHeader_2.54mm:PinHeader_1x03_P2.54mm_Vertical, B.Cu at (136.5, -14.4)
- added JP1: SolderJumper_2_Bridged, Jumper:SolderJumper-2_P1.3mm_Bridged2Bar_Pad1.0x1.5mm, B.Cu at (139.6, 3.98)
- added MX1: MX-NoLED, marbastlib-mx:SW_MX_HS_1u_NOREF, B.Cu at (236.5, 130.2)
- added MX10: MX-NoLED, marbastlib-mx:SW_MX_HS_1u_NOREF, B.Cu at (96.0, 73.0)
- added MX11: MX-NoLED, marbastlib-mx:SW_MX_HS_1u_NOREF, B.Cu at (115.1, 73.0)
- added MX12: MX-NoLED, marbastlib-mx:SW_MX_HS_1u_NOREF, B.Cu at (134.1, 73.0)
- added MX13: MX-NoLED, marbastlib-mx:SW_MX_HS_1u_NOREF, B.Cu at (153.2, 73.0)
- added MX14: MX-NoLED, marbastlib-mx:SW_MX_HS_1u_NOREF, B.Cu at (172.2, 73.0)
- added MX15: MX-NoLED, marbastlib-mx:SW_MX_HS_1u_NOREF, B.Cu at (191.3, 73.0)
- added MX16: MX-NoLED, marbastlib-mx:SW_MX_HS_1u_NOREF, B.Cu at (210.3, 73.0)
- added MX17: MX-NoLED, marbastlib-mx:SW_MX_HS_1u_NOREF, B.Cu at (229.4, 73.0)
- added MX18: MX-NoLED, marbastlib-mx:SW_MX_HS_1u_NOREF, B.Cu at (255.6, 73.0)
- added MX19: MX-NoLED, marbastlib-mx:SW_MX_HS_1u_NOREF, B.Cu at (41.3, 92.1)
- added MX2: MX-NoLED, marbastlib-mx:SW_MX_HS_1u_NOREF, B.Cu at (65.1, 130.2)
- added MX20: MX-NoLED, marbastlib-mx:SW_MX_HS_1u_NOREF, B.Cu at (62.7, 92.1)
- added MX21: MX-NoLED, marbastlib-mx:SW_MX_HS_1u_NOREF, B.Cu at (81.8, 92.1)
- added MX22: MX-NoLED, marbastlib-mx:SW_MX_HS_1u_NOREF, B.Cu at (100.8, 92.1)
- added MX23: MX-NoLED, marbastlib-mx:SW_MX_HS_1u_NOREF, B.Cu at (119.9, 92.1)
- added MX24: MX-NoLED, marbastlib-mx:SW_MX_HS_1u_NOREF, B.Cu at (138.9, 92.1)
- added MX25: MX-NoLED, marbastlib-mx:SW_MX_HS_1u_NOREF, B.Cu at (158.0, 92.1)
- added MX26: MX-NoLED, marbastlib-mx:SW_MX_HS_1u_NOREF, B.Cu at (177.0, 92.1)
- added MX27: MX-NoLED, marbastlib-mx:SW_MX_HS_1u_NOREF, B.Cu at (196.1, 92.1)
- added MX28: MX-NoLED, marbastlib-mx:SW_MX_HS_1u_NOREF, B.Cu at (215.1, 92.1)
- added MX29: MX-NoLED, marbastlib-mx:SW_MX_HS_1u_NOREF, B.Cu at (234.2, 92.1)
- added MX30: MX-NoLED, marbastlib-mx:SW_MX_HS_1u_NOREF, B.Cu at (258.0, 92.1)
- added MX31: MX-NoLED, marbastlib-mx:SW_MX_HS_1u_NOREF, B.Cu at (46.0, 111.1)
- added MX32: MX-NoLED, marbastlib-mx:SW_MX_HS_1u_NOREF, B.Cu at (72.2, 111.1)
- added MX33: MX-NoLED, marbastlib-mx:SW_MX_HS_1u_NOREF, B.Cu at (91.3, 111.1)
- added MX34: MX-NoLED, marbastlib-mx:SW_MX_HS_1u_NOREF, B.Cu at (110.3, 111.1)
- added MX35: MX-NoLED, marbastlib-mx:SW_MX_HS_1u_NOREF, B.Cu at (129.4, 111.1)
- added MX36: MX-NoLED, marbastlib-mx:SW_MX_HS_1u_NOREF, B.Cu at (148.4, 111.1)
- added MX37: MX-NoLED, marbastlib-mx:SW_MX_HS_1u_NOREF, B.Cu at (167.5, 111.1)
- added MX38: MX-NoLED, marbastlib-mx:SW_MX_HS_1u_NOREF, B.Cu at (186.5, 111.1)
- added MX39: MX-NoLED, marbastlib-mx:SW_MX_HS_1u_NOREF, B.Cu at (205.6, 111.1)
- added MX40: MX-NoLED, marbastlib-mx:SW_MX_HS_1u_NOREF, B.Cu at (224.6, 111.1)
- added MX41: MX-NoLED, marbastlib-mx:SW_MX_HS_1u_NOREF, B.Cu at (243.7, 111.1)
- added MX42: MX-NoLED, marbastlib-mx:SW_MX_HS_1u_NOREF, B.Cu at (262.7, 111.1)
- added MX43: MX-NoLED, marbastlib-mx:SW_MX_HS_1u_NOREF, B.Cu at (150.8, 130.2)
- added MX45: MX-NoLED, marbastlib-mx:SW_MX_HS_1u_NOREF, B.Cu at (122.2, 130.2)
- added MX46: MX-NoLED, marbastlib-mx:SW_MX_HS_1u_NOREF, B.Cu at (41.3, 130.2)
- added MX47: MX-NoLED, marbastlib-mx:SW_MX_HS_1u_NOREF, B.Cu at (81.8, 130.2)
- added MX48: MX-NoLED, marbastlib-mx:SW_MX_HS_1u_NOREF, B.Cu at (260.4, 130.2)
- added MX49: MX-NoLED, marbastlib-mx:SW_MX_HS_1u_NOREF, B.Cu at (215.1, 130.2)
- added MX52: MX-NoLED, marbastlib-mx:SW_MX_HS_1u_NOREF, B.Cu at (62.7, 130.2)
- added MX53: MX-NoLED, marbastlib-mx:SW_MX_HS_1u_NOREF, B.Cu at (86.5, 130.2)
- added MX54: MX-NoLED, marbastlib-mx:SW_MX_HS_1u_NOREF, B.Cu at (219.9, 130.2)
- added MX57: MX-NoLED, marbastlib-mx:SW_MX_HS_1u_NOREF, B.Cu at (238.9, 130.2)
- added MX58: MX-NoLED, marbastlib-mx:SW_MX_HS_1u_NOREF, B.Cu at (177.0, 130.2)
- added MX7: MX-NoLED, marbastlib-mx:SW_MX_HS_1u_NOREF, B.Cu at (38.9, 73.0)
- added MX8: MX-NoLED, marbastlib-mx:SW_MX_HS_1u_NOREF, B.Cu at (57.9, 73.0)
- added MX9: MX-NoLED, marbastlib-mx:SW_MX_HS_1u_NOREF, B.Cu at (77.0, 73.0)
- added R10: 470, Resistor_SMD:R_0603_1608Metric, B.Cu at (116.5, -56.1)
- added R11: 470, Resistor_SMD:R_0603_1608Metric, B.Cu at (116.5, -53.5)
- added R12: 1k, Resistor_SMD:R_0402_1005Metric, B.Cu at (236.8, 94.9)
- added R13: -10k, Resistor_SMD:R_0603_1608Metric, B.Cu at (116.5, -51.0)
- added R14: 1k, Resistor_SMD:R_0402_1005Metric, B.Cu at (140.3, -7.79)
- added R2: 5.1k, Resistor_SMD:R_0603_1608Metric, B.Cu at (120.5, -46.0)
- added R4: 5.1k, Resistor_SMD:R_0603_1608Metric, B.Cu at (120.5, -43.5)
- added R5: 5.1k, Resistor_SMD:R_0402_1005Metric, B.Cu at (140.3, -15.7)
- added R6: 27, Resistor_SMD:R_0402_1005Metric, B.Cu at (245.7, 73.8)
- added R7: 27, Resistor_SMD:R_0402_1005Metric, B.Cu at (245.7, 72.8)
- added R9: 470, Resistor_SMD:R_0603_1608Metric, B.Cu at (116.5, -58.6)
- added REF**: STAB_MX_P_6.25u, marbastlib-mx:STAB_MX_P_6.25u, F.Cu at (150.8, 130.2)
- added REF**: STAB_MX_P_3u, marbastlib-mx:STAB_MX_P_3u, F.Cu at (177.0, 130.2)
- added REF**: STAB_MX_P_2u, marbastlib-mx:STAB_MX_P_2u, F.Cu at (122.2, 130.2)
- added SW3: RotaryEncoder_Switch, marbastlib-various:ROT_Alps_EC11E-Switch, F.Cu at (38.9, 73.0)
- added SWD1: Conn_01x03_Female, Connector_PinHeader_2.54mm:PinHeader_1x03_P2.54mm_Vertical, B.Cu at (131.9, -14.4)
- added SWR1: SW_SPST, Keebio-Parts:SW_SPST_TL3342, B.Cu at (131.1, -37.7)
- added SWR2: SW_SPST, Keebio-Parts:SW_SPST_TL3342, B.Cu at (131.1, -30.7)
- added U1: SRV05-4, Package_TO_SOT_SMD:SOT-23-6, B.Cu at (242.5, 74.0)
- added U2: XC6206PxxxMR, Package_TO_SOT_SMD:SOT-23, B.Cu at (139.6, -0.07)
- added U3: RP2040TR7, cipulot_kicad_parts:RP2040-QFN-56, B.Cu at (246.2, 98.4)
- added U4: W25Q128JVS, Package_SO:SOIC-8_5.23x5.23mm_P1.27mm, B.Cu at (125.1, -21.2)
- added Y1: Crystal_GND24_Small, Crystal:Crystal_SMD_3225-4Pin_3.2x2.5mm, B.Cu at (239.6, 95.4)
- J6: footprint Keebio-Parts:USB_C_Receptacle_HRO_TYPE-C-31-M-12 -> Type-C:HRO-TYPE-C-31-M-12-Assembly
- moved G*** 280.7 mm to (79.4, 373.1)
- moved G*** 275.5 mm to (81.8, 368.3)
- moved J6 3.91 mm to (242.5, 60.8)
Routing:
- removed copper zone on F.Cu, net GND
Other:
- outline, holes or cut-outs redrawn

Commit message: set initial positions for components
Parts:
- J6: footprint Type-C:HRO-TYPE-C-31-M-12-Assembly -> Connector_USB:USB_C_Receptacle_HRO_TYPE-C-31-M-12
- moved R13 207.9 mm to (265.9, 93.4)
- moved SWR1 205.6 mm to (265.5, 117.9)
- moved R11 199.1 mm to (26.6, 124.1)
- moved SWR2 197.0 mm to (255.3, 122.3)
- moved R10 194.8 mm to (27.8, 117.4)
- moved R9 194.8 mm to (27.8, 114.9)
- moved J8 193.2 mm to (255.1, 102.9), turned to -90 degrees
- moved C16 191.1 mm to (248.9, 83.0)
- moved D53 191.0 mm to (23.9, 113.0)
- moved D54 191.0 mm to (23.9, 118.6)
- moved D55 191.0 mm to (23.9, 124.1)
- moved C18 183.6 mm to (246.3, 80.2)
- moved U4 182.7 mm to (262.9, 98.8)
- moved C13 178.7 mm to (246.1, 82.4)
- moved C20 178.1 mm to (245.6, 78.2)
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Connections:
- U1 pad 1: D+ -> unconnected-(U1-IO1-Pad1)
- U1 pad 4: unconnected-(U1-IO3-Pad4) -> D-
- U1 pad 6: D- -> D+
Routing:
- net GND: track 0.00 -> 38.1 mm
- net D+: track 0.00 -> 18.9 mm
- net D-: track 0.00 -> 18.8 mm
- net VCC: track 0.00 -> 17.8 mm, vias 0 -> 3
- net Net-(J6-CC2): track 0.00 -> 8.14 mm, vias 0 -> 2
- net Net-(J6-CC1): track 0.00 -> 7.71 mm

Commit message: began routing upper portion, improved placement
Parts:
- removed D57, D58: WS2812B, WS2812B:WS2812B_data-bridgeable
- moved D21 155.0 mm to (294.4, 138.8)
- moved D22 154.2 mm to (288.8, 137.5)
- moved D10 151.8 mm to (281.7, 113.9)
- moved D20 141.9 mm to (284.5, 136.1)
- moved D9 140.5 mm to (273.3, 112.1), turned to -45 degrees
- moved D19 132.2 mm to (278.9, 136.3)
- moved D18 131.4 mm to (227.6, 83.0), turned to 45 degrees
- moved D6 125.0 mm to (222.4, 77.7), turned to 45 degrees
- moved D15 122.1 mm to (225.0, 80.4), turned to 45 degrees
- moved D5 121.8 mm to (219.9, 75.2), turned to 45 degrees
- moved D17 114.2 mm to (233.5, 113.7), turned to 135 degrees
- moved D56 109.6 mm to (53.1, 98.4)
- moved D12 106.9 mm to (225.1, 117.0), turned to -45 degrees
- moved D16 105.1 mm to (227.6, 114.4), turned to -45 degrees
- moved D11 99.6 mm to (222.5, 119.5), turned to -45 degrees
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Routing:
- net Net-(MX2-ROW): track 0.00 -> 163.6 mm
- net Net-(MX47-ROW): track 0.00 -> 140.8 mm
- net ENCB: track 0.00 -> 140.7 mm
- net ROW0: track 0.00 -> 125.9 mm
- net ROW1: track 0.00 -> 123.8 mm
- net Net-(MX42-ROW): track 0.00 -> 88.6 mm
- net LED1: track 0.00 -> 81.2 mm
- net Net-(MX43-ROW): track 0.00 -> 80.9 mm
- net LED3: track 0.00 -> 80.7 mm
- net LED2: track 0.00 -> 80.4 mm
- net ENC_ROW: track 0.00 -> 75.4 mm
- net Net-(MX11-ROW): track 0.00 -> 75.0 mm
- net Net-(MX46-ROW): track 0.00 -> 74.5 mm
- net ENCA: track 0.00 -> 73.1 mm
- net Net-(MX31-ROW): track 0.00 -> 72.7 mm
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
Commit message: updated routing, position of diodes
Parts:
- SW3: moved to B.Cu
- moved J9 170.6 mm to (46.4, 101.0), turned to 0 degrees
- moved D10 161.9 mm to (119.8, 112.0), turned to 45 degrees
- moved D20 157.5 mm to (127.9, 120.0), turned to 45 degrees
- moved D19 154.7 mm to (125.3, 117.5), turned to 45 degrees
- moved D9 151.0 mm to (122.4, 114.6), turned to 45 degrees
- moved JP1 132.1 mm to (230.2, 100.0)
- moved D21 92.3 mm to (204.1, 120.0), turned to 45 degrees
- moved D22 89.6 mm to (201.5, 117.5), turned to 45 degrees
- moved D12 29.5 mm to (196.0, 112.0), turned to 45 degrees
- moved D11 24.5 mm to (198.6, 114.6), turned to 45 degrees
- moved D16 7.00 mm to (234.2, 112.0), turned to 45 degrees
- moved D17 3.39 mm to (236.7, 114.6), turned to 45 degrees
- turned SW3 to 180 degrees
Connections:
- D13 pad 1: Net-(MX23-ROW) -> Net-(MX24-ROW)
- D13 pad 2: Net-(MX24-ROW) -> Net-(MX23-ROW)
- D14 pad 1: Net-(MX25-ROW) -> Net-(MX26-ROW)
- D14 pad 2: Net-(MX26-ROW) -> Net-(MX25-ROW)
- D15 pad 1: Net-(MX27-ROW) -> Net-(MX28-ROW)
- D15 pad 2: Net-(MX28-ROW) -> Net-(MX27-ROW)
- D19 pad 1: Net-(MX46-ROW) -> Net-(MX2-ROW)
- D19 pad 2: Net-(MX2-ROW) -> Net-(MX46-ROW)
- D20 pad 1: Net-(MX47-ROW) -> Net-(MX43-ROW)
- D20 pad 2: Net-(MX43-ROW) -> Net-(MX47-ROW)
- D22 pad 1: Net-(MX58-COL) -> Net-(MX49-COL)
- D22 pad 2: Net-(MX49-COL) -> Net-(MX58-COL)
- D56 pad 2: Net-(D56-DOUT) -> RGB_OUT
- D7 pad 1: Net-(MX19-ROW) -> Net-(MX20-ROW)
- D7 pad 2: Net-(MX20-ROW) -> Net-(MX19-ROW)
- D8 pad 1: Net-(MX21-ROW) -> Net-(MX22-ROW)
- D8 pad 2: Net-(MX22-ROW) -> Net-(MX21-ROW)
- SW3 pad S1: ENC_ROW -> COL0
- SW3 pad S2: COL0 -> ENC_ROW
Routing:
- net +5VD: track 0.00 -> 220.0 mm
- net GND: track 49.7 -> 262.7 mm
- net ENCA: track 73.1 -> 221.9 mm
- net ROW2: track 0.00 -> 124.8 mm
- net COL4: track 0.00 -> 116.7 mm
- net Net-(MX58-COL): track 25.6 -> 129.2 mm, vias 0 -> 2
- net LED3: track 80.7 -> 179.3 mm
- net Net-(MX23-ROW): track 0.00 -> 97.2 mm, vias 0 -> 2
- net COL10: track 0.00 -> 96.3 mm
- net COL1: track 0.00 -> 95.9 mm
- net COL2: track 0.00 -> 94.8 mm
- net COL0: track 0.00 -> 93.4 mm
- net LED2: track 80.4 -> 173.7 mm
- net LED1: track 81.2 -> 172.7 mm
- net COL6: track 0.00 -> 90.7 mm
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
Commit message: finished base routing
Parts:
- removed C10, C11, C12, C9: 0.1uF, Capacitor_SMD:C_0603_1608Metric
- removed C24: 100n, Capacitor_SMD:C_0402_1005Metric
- removed D53, D54, D55: LED, LED_THT:LED_D3.0mm
- removed the G*** at (44.8, 118.7)
- removed R10, R11, R9: 470, Resistor_SMD:R_0603_1608Metric
- added J1: Conn_01x02_Male, Connector_PinHeader_2.54mm:PinHeader_1x02_P2.54mm_Vertical, B.Cu at (37.9, 100.8)
- added J2: Conn_01x02_Male, Connector_PinHeader_2.54mm:PinHeader_1x02_P2.54mm_Vertical, B.Cu at (37.9, 96.4)
- added J3: Conn_01x02_Male, Connector_PinHeader_2.54mm:PinHeader_1x02_P2.54mm_Vertical, B.Cu at (37.9, 98.6)
- moved C17 185.8 mm to (248.8, 78.3), turned to 90 degrees
- moved C19 181.1 mm to (247.3, 78.3), turned to 90 degrees
- moved C15 175.2 mm to (250.4, 78.3), turned to 90 degrees
- moved C25 166.3 mm to (251.2, 92.0), turned to 90 degrees
- moved C26 149.4 mm to (250.2, 92.0), turned to 90 degrees
- moved SWD1 45.5 mm to (233.8, 101.0), turned to 0 degrees
- moved R14 26.5 mm to (266.3, 121.3), turned to -90 degrees
- moved C18 26.5 mm to (230.1, 99.9), turned to 180 degrees
- moved C13 26.2 mm to (230.1, 98.4), turned to 180 degrees
- moved C14 26.1 mm to (230.1, 96.9), turned to 180 degrees
- moved C8 18.6 mm to (245.2, 90.0), turned to -90 degrees
- moved J8 18.0 mm to (269.1, 114.2), turned to 180 degrees
- moved C7 17.0 mm to (247.1, 90.0), turned to -90 degrees
- moved C4 9.15 mm to (245.2, 92.1), turned to 90 degrees
- moved SWR1 8.87 mm to (256.6, 118.0), turned to 90 degrees
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Connections:
- C13 pad 1: +5VD -> +5V
- C14 pad 1: +5VD -> +5V
- C15 pad 1: +5VD -> +5V
- C16 pad 1: +5VD -> +5V
- C17 pad 1: +5VD -> +5V
- C18 pad 1: +5VD -> +5V
- C19 pad 1: +5VD -> +5V
- C20 pad 1: +5VD -> +5V
- J8 pad 2: +5V -> +3V3
- U3 pad 11: unconnected-(U3-GPIO8-Pad11) -> LED2
- U3 pad 12: ROW0 -> LED3
- U3 pad 13: COL8 -> LED1
- U3 pad 14: COL9 -> COL10
- U3 pad 15: ENCA -> ROW2
- U3 pad 16: unconnected-(U3-GPIO13-Pad16) -> COL8
- U3 pad 17: unconnected-(U3-GPIO14-Pad17) -> COL9
- U3 pad 18: unconnected-(U3-GPIO15-Pad18) -> COL7
- U3 pad 2: COL11 -> unconnected-(U3-GPIO0-Pad2)
- U3 pad 27: COL7 -> unconnected-(U3-GPIO16-Pad27)
- U3 pad 28: COL6 -> unconnected-(U3-GPIO17-Pad28)
- U3 pad 29: COL5 -> COL3
- U3 pad 3: ROW1 -> unconnected-(U3-GPIO1-Pad3)
- U3 pad 30: COL4 -> unconnected-(U3-GPIO19-Pad30)
- U3 pad 31: COL3 -> unconnected-(U3-GPIO20-Pad31)
- U3 pad 32: COL2 -> unconnected-(U3-GPIO21-Pad32)
- U3 pad 34: COL1 -> unconnected-(U3-GPIO22-Pad34)
- U3 pad 35: COL0 -> COL2
- U3 pad 36: ENCB -> COL1
- U3 pad 37: LED1 -> COL0
- U3 pad 38: LED2 -> ROW1
- U3 pad 39: LED3 -> ENCA
- U3 pad 4: SDA -> SCL
- U3 pad 40: ROW4 -> ENCB
- U3 pad 41: RGB -> ROW0
- U3 pad 5: SCL -> SDA
- U3 pad 6: ROW2 -> COL11
- U3 pad 7: ROW3 -> COL4
- U3 pad 8: COL10 -> COL5
- U3 pad 9: unconnected-(U3-GPIO7-Pad9) -> COL6
Routing:
- net GND: track 262.7 -> 591.9 mm, vias 0 -> 33
- net COL0: track 93.4 -> 358.1 mm, vias 0 -> 1
- net COL1: track 95.9 -> 331.6 mm, vias 0 -> 2
- net COL2: track 94.8 -> 312.7 mm, vias 0 -> 3
- net COL3: track 54.3 -> 241.5 mm, vias 0 -> 1
- net +3V3: track 0.00 -> 168.8 mm, vias 0 -> 8
- net COL4: track 116.7 -> 276.0 mm, vias 0 -> 3
- net COL5: track 54.2 -> 198.3 mm, vias 0 -> 1
- net COL6: track 90.7 -> 205.5 mm, vias 0 -> 3
- net COL11: track 0.00 -> 89.8 mm
- net LED2: track 173.7 -> 259.9 mm
- net LED1: track 172.7 -> 250.4 mm
- net LED3: track 179.3 -> 254.5 mm
- net QSPI_SS: track 0.00 -> 71.7 mm, vias 0 -> 2
- net COL7: track 54.2 -> 124.6 mm
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- added copper zone on B.Cu, net GND
- added copper zone on F.Cu, net GND
Other:
- board text added: "|| Monorail Steam | Reimagined || By ScatteredDrifter"
- board text removed: "+"
- board text removed: "2023"
- board text removed: "5V GND"
- board text removed: "5VLED"
- board text removed: "GND RGB 5VD"
- board text removed: "GP2 GP3 SDA SCL"
- board text removed: "Monorail Steam Version 2.0"
- board text removed: "RST"
