File: pcb_source/Monorail_Steam_Reduced.kicad_sch (KiCad schematic)
At the start: 131 parts, among them J1 Conn_01x02_Male, J2 Conn_01x02_Male, J3 Conn_01x02_Male, J4 Conn_01x02_Male, J6 USB_C_Receptacle_USB2.0, J8 Conn_01x04_Male, J9 Conn_01x03_Male, SW3 RotaryEncoder_Switch, U1 SRV05-4, U2 XC6206PxxxMR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

Commit message: fix bottom row stabilizer orientation
Connections:
- net at MX48.2 (ROW): now also D21.1 (A); no longer D21.2 (A)
- net at MX1.2 (ROW), MX57.2 (ROW): now also D21.2 (A); no longer D21.1 (A)
Changed lines of the file:
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@@
     )
   )
-  (symbol (lib_id "Diode:BAV70") (at 266.7 119.38 0) (unit 1)
-    (in_bom yes) (on_board yes) (dnp no) (fields_autoplaced)
+  (symbol (lib_id "Diode:BAV70") (at 266.7 119.38 0) (mirror y) (unit 1)
+    (in_bom yes) (on_board yes) (dnp no)
     (property "Reference" "D21" (at 266.7 113.03 0)
       (effects (font (size 1.27 1.27)))
